File: PCBs/Ttl_wlan_radar_v4/processed.kicad_pcb (KiCad board)
At the start: 4 copper layers, 55 x 25 mm, 128 parts, among them P1 CONN_2, P2 CONN_2, P3 CONN_2, P4 CONN_6, Q1 MOS_P_BSS84, U1 SST11LP12, U10 LTC6242, U11 LT6230, U12 MCP4017, U13 USB-MICRO, U14 MKL26Z128VFT4, U15 TSV321RAILT, U16 LM2681, U17 TSV321RAILT, U18 SC189, U19 AAT3220, U2 HMC431LP4, U3 SKY65404, U4 HMC219AMS8, U5 PAT1220-7dB, U7 PAT1220-7dB, U8 MCP1700, X1 8MHz

Commit message: debug rl env and clean data for rl
Connections:
- C15 pad 1: (no net) -> /mcu/3V3A
- C16 pad 1: (no net) -> /mcu/ADC_DP
- C18 pad 2: (no net) -> /mcu/ADC_DM
- C19 pad 1: (no net) -> /mcu/ADC_DM
- C21 pad 2: (no net) -> /VG
- C22 pad 1: (no net) -> /mcu/VBUS
- C24 pad 1: (no net) -> /mcu/PA_DET
- C28 pad 1: (no net) -> /mcu/3V3A
- C38 pad 1: (no net) -> /mcu/3V3A
- C41 pad 1: (no net) -> Net-(C41-Pad1)
- C42 pad 2: (no net) -> /VG
- C43 pad 2: (no net) -> /VG
- C44 pad 1: (no net) -> /mcu/3V3A
- C49 pad 1: (no net) -> /mcu/3V3A
- C52 pad 1: (no net) -> /mcu/~RESET
- P4 pad 1: (no net) -> /mcu/SWD_CLK
- P4 pad 2: (no net) -> /mcu/SWD_DIO
- P4 pad 3: (no net) -> /mcu/~RESET
- P4 pad 4: (no net) -> /mcu/UART_RX
- P4 pad 5: (no net) -> /mcu/UART_TX
- Q1 pad 1: (no net) -> /mcu/PA_EN
- Q1 pad 2: (no net) -> Net-(Q1-Pad2)
- R10 pad 2: (no net) -> /mcu/VBUS
- R12 pad 2: (no net) -> /mcu/I2C_SDA
- R13 pad 2: (no net) -> /mcu/I2C_SCL
- R16 pad 1: (no net) -> /mcu/~RESET
- R17 pad 2: (no net) -> /mcu/DAC_OUT
- R18 pad 2: (no net) -> /VTUNE
- R21 pad 2: (no net) -> /VG
- R22 pad 2: (no net) -> Net-(R22-Pad2)
- R26 pad 2: (no net) -> /VG
- R27 pad 1: (no net) -> /VG
- R3 pad 1: (no net) -> /VG
- R30 pad 2: (no net) -> /VG
- R31 pad 2: (no net) -> /VG
- R32 pad 1: (no net) -> /mcu/3V3A
- R33 pad 1: (no net) -> /VG
- R36 pad 1: (no net) -> /mcu/3V3A
- R4 pad 1: (no net) -> /mcu/ADC_DP
- R40 pad 2: (no net) -> /mcu/PA_EN
- R41 pad 2: (no net) -> Net-(Q1-Pad2)
- R42 pad 2: (no net) -> /VG
- R5 pad 1: (no net) -> Net-(R22-Pad2)
- R6 pad 2: (no net) -> /mcu/ADC_DM
- R8 pad 1: (no net) -> /mcu/ADC_DP
- R9 pad 1: (no net) -> Net-(C41-Pad1)
- R9 pad 2: (no net) -> /VG
- U1 pad 9: (no net) -> /mcu/PA_DET
- U10 pad 10: (no net) -> /mcu/ADC_DM
- U10 pad 14: (no net) -> /VG
- U10 pad 16: (no net) -> /mcu/ADC_DP
- U10 pad 4: (no net) -> /mcu/3V3A
- U11 pad 1: (no net) -> Net-(R22-Pad2)
- U11 pad 4: (no net) -> Net-(C41-Pad1)
- U11 pad 6: (no net) -> /mcu/3V3A
- U12 pad 3: (no net) -> /mcu/I2C_SCL
- U12 pad 4: (no net) -> /mcu/I2C_SDA
- U12 pad 5: (no net) -> Net-(C41-Pad1)
- U13 pad 1: (no net) -> /mcu/VBUS
- U14 pad 10: (no net) -> /mcu/3V3A
- U14 pad 14: (no net) -> /mcu/DAC_OUT
- U14 pad 17: (no net) -> /mcu/SWD_CLK
- U14 pad 18: (no net) -> /mcu/UART_RX
- U14 pad 19: (no net) -> /mcu/UART_TX
- U14 pad 20: (no net) -> /mcu/SWD_DIO
- U14 pad 26: (no net) -> /mcu/~RESET
- U14 pad 27: (no net) -> /mcu/I2C_SCL
- U14 pad 28: (no net) -> /mcu/I2C_SDA
- U14 pad 29: (no net) -> /mcu/PA_EN
- U14 pad 33: (no net) -> /mcu/PA_DET
- U14 pad 6: (no net) -> /mcu/VBUS
- U14 pad 7: (no net) -> /mcu/ADC_DP
- U14 pad 8: (no net) -> /mcu/ADC_DM
- U14 pad 9: (no net) -> /mcu/3V3A
- U15 pad 1: (no net) -> /VTUNE
- U17 pad 4: (no net) -> /VG
- U17 pad 5: (no net) -> /mcu/3V3A
- U19 pad 2: (no net) -> /mcu/3V3A
- U2 pad 22: (no net) -> /VTUNE
Routing:
- net /VG: track 0.00 -> 56.4 mm, vias 0 -> 6
- net /mcu/3V3A: track 0.00 -> 50.4 mm, vias 0 -> 8
- net /mcu/PA_DET: track 0.00 -> 45.9 mm, vias 0 -> 3
- net /mcu/I2C_SDA: track 0.00 -> 38.4 mm, vias 0 -> 5
- net /mcu/UART_TX: track 0.00 -> 38.2 mm, vias 0 -> 1
- net /mcu/UART_RX: track 0.00 -> 35.5 mm, vias 0 -> 1
- net /mcu/I2C_SCL: track 0.00 -> 34.9 mm, vias 0 -> 2
- net /mcu/PA_EN: track 0.00 -> 27.8 mm, vias 0 -> 2
- net /mcu/~RESET: track 0.00 -> 27.4 mm, vias 0 -> 2
- net /mcu/SWD_DIO: track 0.00 -> 24.0 mm, vias 0 -> 1
- net /mcu/VBUS: track 0.00 -> 21.6 mm, vias 0 -> 2
- net /mcu/DAC_OUT: track 0.00 -> 15.7 mm, vias 0 -> 2
- net /mcu/SWD_CLK: track 0.00 -> 15.5 mm, vias 0 -> 1
- net /mcu/ADC_DP: track 0.00 -> 15.3 mm, vias 0 -> 2
- net /mcu/ADC_DM: track 0.00 -> 13.4 mm, vias 0 -> 3
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