File: PCBs/kitspace_12V5A_breakout/processed.kicad_pcb (KiCad board)
At the start: 2 copper layers, 48.5 x 45.5 mm, 18 parts, among them J1 Barrel_Jack_Switch, J10 Conn_01x02, J2 Conn_01x02, J3 Conn_01x02, J4 Conn_01x02, J5 Conn_01x02, J6 Conn_01x02, J7 Conn_01x02, J8 Conn_01x02, J9 Conn_01x02

Commit message: recheck all circuits and clean up fill zone by rerouting the nets using freerouting and manually
Parts:
- removed the REF** at (120.0, 81.5)
- removed the REF** at (78.5, 81.5)
- removed the REF** at (78.5, 43.0)
- added REF**_2: MountingHole_3.2mm_M3_DIN965, MountingHole:MountingHole_3.2mm_M3_DIN965, F.Cu at (78.5, 43.0)
- added REF**_3: MountingHole_3.2mm_M3_DIN965, MountingHole:MountingHole_3.2mm_M3_DIN965, F.Cu at (78.5, 81.5)
- added REF**_4: MountingHole_3.2mm_M3_DIN965, MountingHole:MountingHole_3.2mm_M3_DIN965, F.Cu at (120.0, 81.5)
- renumbered REF** to REF**_5
Connections:
- J1 pad 2: (no net) -> GND
- J1 pad 3: (no net) -> GND
- J10 pad 1: (no net) -> GND
- J2 pad 1: (no net) -> GND
- J3 pad 1: (no net) -> GND
- J4 pad 1: (no net) -> GND
- J5 pad 1: (no net) -> GND
- J6 pad 1: (no net) -> GND
- J7 pad 1: (no net) -> GND
- J8 pad 1: (no net) -> GND
- J9 pad 1: (no net) -> GND
- POW pad 1: (no net) -> GND
Routing:
- net GND: track 0.00 -> 108.5 mm
- net +12V: track 116.8 -> 125.2 mm
