File: PCBs/kitspace_BalthazarKeyboard3-keycaps/processed.kicad_pcb (KiCad board)
At the start: 4 copper layers, 290.6 x 127 mm, 199 parts, among them J1 USB, J2 USB_B_Micro, J3 PS2 touchpad, J4 ISP, J5 I2C, SW1 ESC, SW10 2, SW11 3, SW12 4, SW13 5, SW14 6, SW15 TAB, SW16 Q, SW17 W, SW18 E, SW19 R, SW2 F1, SW20 T, SW21 Y, SW22 CAPS, SW23 A, SW24 S, SW25 D, SW26 F, SW27 G, SW28 H, SW29 SHIFT, SW3 F2, SW30 NUBS, SW31 Z, SW32 X, SW33 C, SW34 V, SW35 B, SW36 CTRL, SW37 ALT, SW38 GUI, SW39 SPACE, SW4 F3, SW40 SPACE, SW42 LEFT, SW43 DOWN, SW44 RIGHT, SW45 F7, SW46 F8, SW47 F9, SW48 F10, SW49 F11, SW5 F4, SW50 F12, SW51 PRTSCR, SW52 7, SW53 8, SW54 9, SW55 0, SW56 MINUS, SW57 EQUAL, SW58 DELETE, SW59 U, SW6 F5, SW60 I, SW61 O, SW62 P, SW63 LBRC, SW64 RBRC, SW65 BACKSPACE, SW66 J, SW67 K, SW68 L, SW69 SCLN, SW7 F6, SW70 QUOTE, SW71 NUHS, SW72 ENTER, SW73 N, SW74 M, SW75 COMMA, SW76 DOT, SW77 SLASH, SW78 UP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

Commit message: recheck all circuits and clean up fill zone by rerouting the nets using freerouting and manually
Parts:
- renumbered H2 to H2_2, H3 to H3_2, H3 to H3_3, H3 to H3_4, H4 to H4_2
Connections:
- C1 pad 1: (no net) -> Net-(C1-Pad1)
- C1 pad 2: (no net) -> GND
- C2 pad 1: (no net) -> GND
- C2 pad 2: (no net) -> Vcc
- C3 pad 1: (no net) -> GND
- C3 pad 2: (no net) -> Vcc
- C4 pad 1: (no net) -> Net-(C4-Pad1)
- C4 pad 2: (no net) -> GND
- C5 pad 1: (no net) -> Net-(C5-Pad1)
- C5 pad 2: (no net) -> GND
- C6 pad 1: (no net) -> Net-(C6-Pad1)
- C6 pad 2: (no net) -> GND
- C7 pad 1: (no net) -> GND
- C7 pad 2: (no net) -> Vcc
- C8 pad 1: (no net) -> GND
- C8 pad 2: (no net) -> Vcc
- C9 pad 1: (no net) -> GND
- C9 pad 2: (no net) -> Vcc
- D1 pad 1: (no net) -> col1
- D1 pad 2: (no net) -> Net-(D1-Pad2)
- D10 pad 1: (no net) -> col2
- D10 pad 2: (no net) -> Net-(D10-Pad2)
- D11 pad 1: (no net) -> col2
- D11 pad 2: (no net) -> Net-(D11-Pad2)
- D12 pad 1: (no net) -> col2
- D12 pad 2: (no net) -> Net-(D12-Pad2)
- D13 pad 1: (no net) -> col2
- D13 pad 2: (no net) -> Net-(D13-Pad2)
- D14 pad 1: (no net) -> col2
- D15 pad 1: (no net) -> col3
- D15 pad 2: (no net) -> Net-(D15-Pad2)
- D16 pad 1: (no net) -> col3
- D16 pad 2: (no net) -> Net-(D16-Pad2)
- D17 pad 1: (no net) -> col3
- D17 pad 2: (no net) -> Net-(D17-Pad2)
- D18 pad 1: (no net) -> col3
- D18 pad 2: (no net) -> Net-(D18-Pad2)
- D19 pad 2: (no net) -> Net-(D19-Pad2)
- D2 pad 1: (no net) -> col1
- D2 pad 2: (no net) -> Net-(D2-Pad2)
- D20 pad 2: (no net) -> Net-(D20-Pad2)
- D21 pad 1: (no net) -> col3
- D22 pad 1: (no net) -> GND
- D22 pad 2: (no net) -> Net-(D22-Pad2)
- D23 pad 1: (no net) -> col4
- D23 pad 2: (no net) -> Net-(D23-Pad2)
- D24 pad 1: (no net) -> col4
- D24 pad 2: (no net) -> Net-(D24-Pad2)
- D25 pad 1: (no net) -> col4
- D25 pad 2: (no net) -> Net-(D25-Pad2)
- D26 pad 1: (no net) -> col4
- D26 pad 2: (no net) -> Net-(D26-Pad2)
- D27 pad 1: (no net) -> col4
- D27 pad 2: (no net) -> Net-(D27-Pad2)
- D28 pad 1: (no net) -> col4
- D28 pad 2: (no net) -> Net-(D28-Pad2)
- D29 pad 1: (no net) -> col4
- D29 pad 2: (no net) -> Net-(D29-Pad2)
- D3 pad 1: (no net) -> col1
- D3 pad 2: (no net) -> Net-(D3-Pad2)
- D30 pad 1: (no net) -> col5
- D30 pad 2: (no net) -> Net-(D30-Pad2)
- D31 pad 1: (no net) -> col5
- D31 pad 2: (no net) -> Net-(D31-Pad2)
- D32 pad 1: (no net) -> col5
- D32 pad 2: (no net) -> Net-(D32-Pad2)
- D33 pad 2: (no net) -> Net-(D33-Pad2)
- D35 pad 2: (no net) -> Net-(D35-Pad2)
- D36 pad 1: (no net) -> col5
- D36 pad 2: (no net) -> Net-(D36-Pad2)
- D37 pad 1: (no net) -> GND
- D37 pad 2: (no net) -> Net-(D37-Pad2)
- D38 pad 1: (no net) -> col6
- D38 pad 2: (no net) -> Net-(D38-Pad2)
- D39 pad 1: (no net) -> col6
- D39 pad 2: (no net) -> Net-(D39-Pad2)
- D4 pad 1: (no net) -> col1
- D4 pad 2: (no net) -> Net-(D4-Pad2)
- D40 pad 1: (no net) -> col6
- D40 pad 2: (no net) -> Net-(D40-Pad2)
- D41 pad 1: (no net) -> col6
- D42 pad 1: (no net) -> col6
- D43 pad 1: (no net) -> col6
- D44 pad 1: (no net) -> col6
- D45 pad 2: (no net) -> Net-(D45-Pad2)
- D46 pad 1: (no net) -> col11
- D46 pad 2: (no net) -> Net-(D46-Pad2)
- D47 pad 1: (no net) -> col11
- D47 pad 2: (no net) -> Net-(D47-Pad2)
- D48 pad 1: (no net) -> col11
- D49 pad 1: (no net) -> col11
- D49 pad 2: (no net) -> Net-(D49-Pad2)
- D5 pad 1: (no net) -> col1
- D5 pad 2: (no net) -> Net-(D5-Pad2)
- D50 pad 2: (no net) -> Net-(D50-Pad2)
- D51 pad 1: (no net) -> col11
- D51 pad 2: (no net) -> Net-(D51-Pad2)
- D53 pad 1: (no net) -> col10
- D54 pad 1: (no net) -> col10
- D55 pad 1: (no net) -> col10
- D55 pad 2: (no net) -> Net-(D55-Pad2)
- D56 pad 1: (no net) -> col10
- D56 pad 2: (no net) -> Net-(D56-Pad2)
- D57 pad 2: (no net) -> Net-(D57-Pad2)
- D58 pad 1: (no net) -> col10
- D58 pad 2: (no net) -> Net-(D58-Pad2)
- D6 pad 1: (no net) -> col1
- D6 pad 2: (no net) -> Net-(D6-Pad2)
- D60 pad 1: (no net) -> col9
- D61 pad 1: (no net) -> col9
- D62 pad 1: (no net) -> col9
- D63 pad 1: (no net) -> col9
- D63 pad 2: (no net) -> Net-(D63-Pad2)
- D64 pad 1: (no net) -> col9
- D64 pad 2: (no net) -> Net-(D64-Pad2)
- D65 pad 1: (no net) -> col9
- D65 pad 2: (no net) -> Net-(D65-Pad2)
- D66 pad 1: (no net) -> col8
- D67 pad 1: (no net) -> col8
- D68 pad 1: (no net) -> col8
- D69 pad 2: (no net) -> Net-(D69-Pad2)
- D70 pad 1: (no net) -> col8
- D71 pad 1: (no net) -> col8
- D72 pad 1: (no net) -> col8
- D73 pad 1: (no net) -> col7
- D73 pad 2: (no net) -> Net-(D73-Pad2)
- D74 pad 2: (no net) -> Net-(D74-Pad2)
- D75 pad 1: (no net) -> col7
- D75 pad 2: (no net) -> Net-(D75-Pad2)
- D76 pad 1: (no net) -> col7
- D76 pad 2: (no net) -> Net-(D76-Pad2)
- D77 pad 2: (no net) -> Net-(D77-Pad2)
- D78 pad 1: (no net) -> col7
- D78 pad 2: (no net) -> Net-(D78-Pad2)
- D79 pad 2: (no net) -> Net-(D79-Pad2)
- D8 pad 1: (no net) -> col2
- D8 pad 2: (no net) -> Net-(D8-Pad2)
- D9 pad 1: (no net) -> col2
- D9 pad 2: (no net) -> Net-(D9-Pad2)
- H1 pad 1: (no net) -> GND
- H2 pad 1: (no net) -> GND
- H2_2 pad 1: (no net) -> GND
- H3 pad 1: (no net) -> GND
- H3_2 pad 1: (no net) -> GND
- H3_3 pad 1: (no net) -> GND
- H3_4 pad 1: (no net) -> GND
- H4 pad 1: (no net) -> GND
- H4_2 pad 1: (no net) -> GND
- J1 pad 4: (no net) -> GND
- J2 pad 1: (no net) -> Net-(J1-Pad1)
- J2 pad 5: (no net) -> GND
- J2 pad 6: (no net) -> GND
- J3 pad 1: (no net) -> Vcc
- J3 pad 4: (no net) -> GND
- J4 pad 4: (no net) -> RST
- J4 pad 5: (no net) -> Vcc
- J4 pad 6: (no net) -> GND
- J5 pad 1: (no net) -> GND
- J5 pad 2: (no net) -> Vcc
- L1 pad 1: (no net) -> Vcc
- R17 pad 1: (no net) -> Net-(D22-Pad2)
- R18 pad 1: (no net) -> Vcc
- R18 pad 2: (no net) -> PS2clock
- R19 pad 1: (no net) -> Vcc
- R19 pad 2: (no net) -> PS2data
- R3 pad 1: (no net) -> Net-(J1-Pad2)
- R4 pad 2: (no net) -> Net-(R4-Pad2)
- R7 pad 1: (no net) -> Vcc
- R7 pad 2: (no net) -> RST
- R8 pad 1: (no net) -> Net-(D37-Pad2)
- R8 pad 2: (no net) -> Vcc
- SW1 pad 1: (no net) -> row1
- SW1 pad 2: (no net) -> Net-(D1-Pad2)
- SW10 pad 1: (no net) -> row3
- SW10 pad 2: (no net) -> Net-(D10-Pad2)
- SW11 pad 1: (no net) -> row4
- SW11 pad 2: (no net) -> Net-(D11-Pad2)
- SW12 pad 1: (no net) -> row5
- SW12 pad 2: (no net) -> Net-(D12-Pad2)
- SW13 pad 1: (no net) -> row6
- SW13 pad 2: (no net) -> Net-(D13-Pad2)
- SW14 pad 1: (no net) -> row7
- SW15 pad 1: (no net) -> row1
- SW15 pad 2: (no net) -> Net-(D15-Pad2)
- SW16 pad 1: (no net) -> row2
- SW16 pad 2: (no net) -> Net-(D16-Pad2)
- SW17 pad 1: (no net) -> row3
- SW17 pad 2: (no net) -> Net-(D17-Pad2)
- SW18 pad 1: (no net) -> row4
- SW18 pad 2: (no net) -> Net-(D18-Pad2)
- SW19 pad 1: (no net) -> row5
- SW19 pad 2: (no net) -> Net-(D19-Pad2)
- SW2 pad 1: (no net) -> row2
- SW2 pad 2: (no net) -> Net-(D2-Pad2)
- SW20 pad 1: (no net) -> row6
- SW20 pad 2: (no net) -> Net-(D20-Pad2)
- SW21 pad 1: (no net) -> row7
- SW22 pad 1: (no net) -> row1
- SW22 pad 2: (no net) -> Net-(D23-Pad2)
- SW23 pad 1: (no net) -> row2
- SW23 pad 2: (no net) -> Net-(D24-Pad2)
- SW24 pad 1: (no net) -> row3
- SW24 pad 2: (no net) -> Net-(D25-Pad2)
- SW25 pad 1: (no net) -> row4
- SW25 pad 2: (no net) -> Net-(D26-Pad2)
- SW26 pad 1: (no net) -> row5
- SW26 pad 2: (no net) -> Net-(D27-Pad2)
- SW27 pad 1: (no net) -> row6
- SW27 pad 2: (no net) -> Net-(D28-Pad2)
- SW28 pad 1: (no net) -> row7
- SW28 pad 2: (no net) -> Net-(D29-Pad2)
- SW29 pad 1: (no net) -> row1
- SW29 pad 2: (no net) -> Net-(D30-Pad2)
- SW3 pad 1: (no net) -> row3
- SW3 pad 2: (no net) -> Net-(D3-Pad2)
- SW30 pad 1: (no net) -> row2
- SW30 pad 2: (no net) -> Net-(D31-Pad2)
- SW31 pad 1: (no net) -> row3
- SW31 pad 2: (no net) -> Net-(D32-Pad2)
- SW32 pad 1: (no net) -> row4
- SW32 pad 2: (no net) -> Net-(D33-Pad2)
- SW33 pad 1: (no net) -> row5
- SW34 pad 1: (no net) -> row6
- SW34 pad 2: (no net) -> Net-(D35-Pad2)
- SW35 pad 1: (no net) -> row7
- SW35 pad 2: (no net) -> Net-(D36-Pad2)
- SW36 pad 1: (no net) -> row1
- SW36 pad 2: (no net) -> Net-(D38-Pad2)
- SW37 pad 1: (no net) -> row2
- SW37 pad 2: (no net) -> Net-(D39-Pad2)
- SW38 pad 1: (no net) -> row3
- SW38 pad 2: (no net) -> Net-(D40-Pad2)
- SW39 pad 1: (no net) -> row4
- SW4 pad 1: (no net) -> row4
- SW4 pad 2: (no net) -> Net-(D4-Pad2)
- SW40 pad 1: (no net) -> row4
- SW40 pad 2: (no net) -> Net-(D41-Pad2)
- SW42 pad 1: (no net) -> row5
- SW43 pad 1: (no net) -> row6
- SW44 pad 1: (no net) -> row7
- SW45 pad 1: (no net) -> row1
- SW45 pad 2: (no net) -> Net-(D45-Pad2)
- SW46 pad 1: (no net) -> row2
- SW46 pad 2: (no net) -> Net-(D46-Pad2)
- SW47 pad 1: (no net) -> row3
- SW47 pad 2: (no net) -> Net-(D47-Pad2)
- SW48 pad 1: (no net) -> row4
- SW49 pad 1: (no net) -> row5
- SW49 pad 2: (no net) -> Net-(D49-Pad2)
- SW5 pad 1: (no net) -> row5
- SW5 pad 2: (no net) -> Net-(D5-Pad2)
- SW50 pad 1: (no net) -> row6
- SW50 pad 2: (no net) -> Net-(D50-Pad2)
- SW51 pad 1: (no net) -> row7
- SW51 pad 2: (no net) -> Net-(D51-Pad2)
- SW52 pad 1: (no net) -> row1
- SW53 pad 1: (no net) -> row2
- SW54 pad 1: (no net) -> row3
- SW55 pad 1: (no net) -> row4
- SW55 pad 2: (no net) -> Net-(D55-Pad2)
- SW56 pad 1: (no net) -> row5
- SW56 pad 2: (no net) -> Net-(D56-Pad2)
- SW57 pad 1: (no net) -> row6
- SW57 pad 2: (no net) -> Net-(D57-Pad2)
- SW58 pad 1: (no net) -> row7
- SW58 pad 2: (no net) -> Net-(D58-Pad2)
- SW59 pad 1: (no net) -> row1
- SW6 pad 1: (no net) -> row6
- SW6 pad 2: (no net) -> Net-(D6-Pad2)
- SW60 pad 1: (no net) -> row2
- SW61 pad 1: (no net) -> row3
- SW62 pad 1: (no net) -> row4
- SW63 pad 1: (no net) -> row5
- SW63 pad 2: (no net) -> Net-(D63-Pad2)
- SW64 pad 1: (no net) -> row6
- SW64 pad 2: (no net) -> Net-(D64-Pad2)
- SW65 pad 1: (no net) -> row7
- SW65 pad 2: (no net) -> Net-(D65-Pad2)
- SW66 pad 1: (no net) -> row1
- SW67 pad 1: (no net) -> row2
- SW68 pad 1: (no net) -> row3
- SW69 pad 1: (no net) -> row4
- SW69 pad 2: (no net) -> Net-(D69-Pad2)
- SW7 pad 1: (no net) -> row7
- SW70 pad 1: (no net) -> row5
- SW71 pad 1: (no net) -> row6
- SW72 pad 1: (no net) -> row7
- SW73 pad 1: (no net) -> row1
- SW73 pad 2: (no net) -> Net-(D73-Pad2)
- SW74 pad 1: (no net) -> row2
- SW74 pad 2: (no net) -> Net-(D74-Pad2)
- SW75 pad 1: (no net) -> row3
- SW75 pad 2: (no net) -> Net-(D75-Pad2)
- SW76 pad 1: (no net) -> row4
- SW76 pad 2: (no net) -> Net-(D76-Pad2)
- SW77 pad 1: (no net) -> row5
- SW77 pad 2: (no net) -> Net-(D77-Pad2)
- SW78 pad 1: (no net) -> row6
- SW78 pad 2: (no net) -> Net-(D78-Pad2)
- SW79 pad 1: (no net) -> row7
- SW79 pad 2: (no net) -> Net-(D79-Pad2)
- SW8 pad 1: (no net) -> row1
- SW8 pad 2: (no net) -> Net-(D8-Pad2)
- SW80 pad 1: (no net) -> GND
- SW80 pad 2: (no net) -> RST
- SW9 pad 1: (no net) -> row2
- SW9 pad 2: (no net) -> Net-(D9-Pad2)
- U1 pad 1: (no net) -> row7
- U1 pad 13: (no net) -> RST
- U1 pad 14: (no net) -> Vcc
- U1 pad 15: (no net) -> GND
- U1 pad 16: (no net) -> Net-(C5-Pad1)
- U1 pad 17: (no net) -> Net-(C6-Pad1)
- U1 pad 2: (no net) -> Vcc
- U1 pad 23: (no net) -> GND
- U1 pad 24: (no net) -> Vcc
- U1 pad 28: (no net) -> col6
- U1 pad 30: (no net) -> col4
- U1 pad 32: (no net) -> col2
- U1 pad 34: (no net) -> Vcc
- U1 pad 35: (no net) -> GND
- U1 pad 36: (no net) -> row6
- U1 pad 37: (no net) -> row5
- U1 pad 38: (no net) -> row4
- U1 pad 39: (no net) -> row3
- U1 pad 4: (no net) -> Net-(R4-Pad2)
- U1 pad 40: (no net) -> row2
- U1 pad 41: (no net) -> row1
- U1 pad 42: (no net) -> Net-(C4-Pad1)
- U1 pad 43: (no net) -> GND
- U1 pad 44: (no net) -> Vcc
- U1 pad 5: (no net) -> GND
- U1 pad 6: (no net) -> Net-(C1-Pad1)
- U1 pad 7: (no net) -> Vcc
- Y1 pad 1: (no net) -> Net-(C5-Pad1)
- Y1 pad 2: (no net) -> GND
- Y1 pad 3: (no net) -> Net-(C6-Pad1)
- Y1 pad 4: (no net) -> GND
Routing:
- net GND: track 0.00 -> 886.3 mm, vias 0 -> 5
- net row4: track 0.00 -> 531.0 mm
- net col6: track 0.00 -> 441.7 mm
- net row3: track 0.00 -> 432.6 mm, vias 0 -> 2
- net row5: track 0.00 -> 410.5 mm, vias 0 -> 2
- net row7: track 0.00 -> 391.1 mm, vias 0 -> 3
- net row1: track 0.00 -> 390.4 mm, vias 0 -> 1
- net row6: track 0.00 -> 384.5 mm
- net row2: track 0.00 -> 379.7 mm, vias 0 -> 2
- net col4: track 0.00 -> 242.6 mm, vias 0 -> 2
- net col2: track 0.00 -> 190.5 mm, vias 0 -> 2
- net col5: track 161.3 -> 330.5 mm, vias 0 -> 2
- net Vcc: track 0.00 -> 155.8 mm, vias 0 -> 1
- net col3: track 87.7 -> 237.3 mm, vias 1 -> 2
- net col9: track 63.7 -> 211.0 mm
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