File: PCBs/kitspace_flypi_v2/processed.kicad_pcb (KiCad board)
At the start: 2 copper layers, 76 x 85 mm, 35 parts, among them CON1 BARREL_JACK, J1 USB_A, P1 D1, P10 A2, P11 A3, P12 I2C 1, P13 I2C 2, P14 12V, P15 UART, P2 D2, P3 D3, P4 D4, P5 D5, P6 D6, P7 D7, P8 D8, P9 A1, U1 LM2596, U2 LM2596, U3 ESP32-DEVKITC-32D

Commit message: recheck all circuits and clean up fill zone by rerouting the nets using freerouting and manually
Parts:
- removed ?: , 
- removed ? (x4): , Mounting_Holes:MountingHole_3.2mm_M3_DIN965
- added Noname_3: , Mounting_Holes:MountingHole_3.2mm_M3_DIN965, F.Cu at (206.5, 64.5)
- added Noname_4: , Mounting_Holes:MountingHole_3.2mm_M3_DIN965, F.Cu at (139.5, 64.5)
- added Noname_5: , , F.Cu at (145.5, 79.0)
- added None_1: , Mounting_Holes:MountingHole_3.2mm_M3_DIN965, F.Cu at (139.5, 140.5)
- added None_2: , Mounting_Holes:MountingHole_3.2mm_M3_DIN965, F.Cu at (206.5, 140.5)
- Noname_1, Noname_2: renamed from  
Connections:
- C1 pad 1: (no net) -> Net-(C1-Pad1)
- C2 pad 1: (no net) -> Net-(C2-Pad1)
- C2 pad 2: (no net) -> GND
- C3 pad 1: (no net) -> Net-(C1-Pad1)
- C3 pad 2: (no net) -> GND
- C4 pad 2: (no net) -> GND
- CON1 pad 1: (no net) -> Net-(C1-Pad1)
- CON1 pad 2: (no net) -> GND
- CON1 pad 3: (no net) -> GND
- D1 pad 2: (no net) -> GND
- D2 pad 2: (no net) -> GND
- J1 pad 1: (no net) -> Net-(C2-Pad1)
- J1 pad 2: (no net) -> Net-(J1-Pad2)
- J1 pad 3: (no net) -> Net-(J1-Pad3)
- J1 pad 4: (no net) -> GND
- J1 pad 5: (no net) -> GND
- L1 pad 2: (no net) -> Net-(C2-Pad1)
- P1 pad 1: (no net) -> +5V
- P1 pad 2: (no net) -> GND
- P10 pad 1: (no net) -> +5V
- P11 pad 1: (no net) -> +5V
- P12 pad 1: (no net) -> +5V
- P12 pad 2: (no net) -> GND
- P13 pad 1: (no net) -> +5V
- P13 pad 2: (no net) -> GND
- P14 pad 1: (no net) -> Net-(C1-Pad1)
- P14 pad 2: (no net) -> GND
- P14 pad 3: (no net) -> Net-(P14-Pad3)
- P14 pad 4: (no net) -> Net-(P14-Pad4)
- P15 pad 1: (no net) -> +5V
- P15 pad 2: (no net) -> GND
- P2 pad 1: (no net) -> +5V
- P2 pad 2: (no net) -> GND
- P3 pad 1: (no net) -> +5V
- P3 pad 2: (no net) -> GND
- P4 pad 1: (no net) -> +5V
- P4 pad 2: (no net) -> GND
- P5 pad 1: (no net) -> +5V
- P5 pad 2: (no net) -> GND
- P6 pad 1: (no net) -> +5V
- P6 pad 2: (no net) -> GND
- P7 pad 1: (no net) -> +5V
- P7 pad 2: (no net) -> GND
- P8 pad 1: (no net) -> +5V
- P8 pad 2: (no net) -> GND
- P9 pad 1: (no net) -> +5V
- P9 pad 2: (no net) -> GND
- U1 pad 1: (no net) -> Net-(C1-Pad1)
- U1 pad 3: (no net) -> GND
- U1 pad 4: (no net) -> Net-(C2-Pad1)
- U1 pad 5: (no net) -> GND
- U2 pad 1: (no net) -> Net-(C1-Pad1)
- U2 pad 3: (no net) -> GND
- U2 pad 4: (no net) -> +5V
- U2 pad 5: (no net) -> GND
- U3 pad 1: (no net) -> Net-(U3-Pad1)
- U3 pad 14: (no net) -> GND
- U3 pad 19: (no net) -> +5V
- U3 pad 2: (no net) -> Net-(U3-Pad2)
- U3 pad 20: (no net) -> GND
- U3 pad 21: (no net) -> Net-(U3-Pad21)
- U3 pad 22: (no net) -> Net-(U3-Pad22)
- U3 pad 25: (no net) -> Net-(U3-Pad25)
- U3 pad 26: (no net) -> GND
- U3 pad 38: (no net) -> Net-(U3-Pad38)
Routing:
- net GND: track 18.6 -> 359.0 mm
- net +5V: track 17.4 -> 250.9 mm
- net Net-(C1-Pad1): track 0.00 -> 86.5 mm
- net Net-(C2-Pad1): track 0.00 -> 43.5 mm
- net Net-(D1-Pad1): track 27.2 -> 30.6 mm
- net Net-(D2-Pad1): track 27.2 -> 29.9 mm
