File: PCBs/kitspace_level_shifter/processed.kicad_pcb (KiCad board)
At the start: 2 copper layers, 45.5 x 48.5 mm, 25 parts, among them J1 Conn_01x04, J2 Conn_01x04, J3 Conn_01x02, J4 Conn_01x02, J5 Conn_01x02, J6 Conn_01x02, Q1 2N7000, Q2 2N7000, Q3 2N7000, Q4 2N7000

Commit message: recheck all circuits and clean up fill zone by rerouting the nets using freerouting and manually
Parts:
- renumbered REF** to REF**_2, REF** to REF**_3, REF** to REF**_4
Connections:
- J1 pad 1: (no net) -> d2_l
- J1 pad 2: (no net) -> d1_l
- J1 pad 3: (no net) -> +5V
- J1 pad 4: (no net) -> GND
- J2 pad 1: (no net) -> d4_l
- J2 pad 2: (no net) -> d3_l
- J2 pad 3: (no net) -> +5V
- J2 pad 4: (no net) -> GND
- J3 pad 2: (no net) -> GND
- J4 pad 2: (no net) -> GND
- J5 pad 2: (no net) -> GND
- J6 pad 2: (no net) -> GND
- Q1 pad 1: (no net) -> d1_l
- Q1 pad 2: (no net) -> +3V3
- Q2 pad 1: (no net) -> d2_l
- Q2 pad 2: (no net) -> +3V3
- Q3 pad 1: (no net) -> d3_l
- Q3 pad 2: (no net) -> +3V3
- Q4 pad 1: (no net) -> d4_l
- Q4 pad 2: (no net) -> +3V3
- R1 pad 1: (no net) -> +3V3
- R1 pad 2: (no net) -> +5V
- R10 pad 1: (no net) -> +5V
- R2 pad 1: (no net) -> GND
- R2 pad 2: (no net) -> +3V3
- R3 pad 1: (no net) -> +3V3
- R3 pad 2: (no net) -> d1_l
- R4 pad 1: (no net) -> +3V3
- R4 pad 2: (no net) -> d2_l
- R5 pad 1: (no net) -> +3V3
- R5 pad 2: (no net) -> d3_l
- R6 pad 1: (no net) -> +3V3
- R6 pad 2: (no net) -> d4_l
- R7 pad 1: (no net) -> +5V
- R8 pad 1: (no net) -> +5V
- R9 pad 1: (no net) -> +5V
Routing:
- net +3V3: track 0.00 -> 96.6 mm
- net GND: track 0.00 -> 92.0 mm
- net +5V: track 0.00 -> 72.2 mm
- net d1_l: track 0.00 -> 34.5 mm
- net d4_l: track 0.00 -> 30.6 mm
- net d3_l: track 0.00 -> 30.3 mm
- net d2_l: track 0.00 -> 29.2 mm
