File: PCBs/kitspace_BQ25570_Harvester/processed.kicad_pcb (KiCad board)
At the start: 2 copper layers, 12.7 x 20.8 mm, 20 parts, among them P1 INPUT, P2 LIPO, P3 LOAD, U1 TI_BQ25570

Commit message: recheck all circuits and clean up fill zone by rerouting the nets using freerouting and manually
Connections:
- C1 pad 2: (no net) -> GND
- C2 pad 2: (no net) -> GND
- C3 pad 2: (no net) -> GND
- C4 pad 2: (no net) -> GND
- C5 pad 2: (no net) -> GND
- C6 pad 2: (no net) -> GND
- C7 pad 2: (no net) -> GND
- L1 pad 1: (no net) -> /VIN
- L1 pad 2: (no net) -> Net-(L1-Pad2)
- P1 pad 2: (no net) -> GND
- P2 pad 1: (no net) -> +BATT
- P2 pad 2: (no net) -> GND
- P3 pad 2: (no net) -> GND
- R2 pad 2: (no net) -> GND
- R5 pad 2: (no net) -> GND
- R7 pad 2: (no net) -> GND
- U1 pad 1: (no net) -> GND
- U1 pad 15: (no net) -> GND
- U1 pad 17: (no net) -> GND
- U1 pad 18: (no net) -> +BATT
- U1 pad 20: (no net) -> Net-(L1-Pad2)
- U1 pad 21: (no net) -> GND
- U1 pad 5: (no net) -> GND
- U1 pad 9: (no net) -> GND
Routing:
- net GND: track 0.00 -> 79.7 mm, vias 0 -> 5
- net +BATT: track 0.00 -> 26.9 mm
- net Net-(L1-Pad2): track 0.00 -> 5.71 mm
