File: PCBs/kitspace_PSLab/processed.kicad_pcb (KiCad board)
At the start: 4 copper layers, 72.9 x 53.6 mm, 144 parts, among them CON1 USB-MICRO-B, J1 V+, J10 I2C-I, J11 I2C-II, J12 Ex-II, J2 GND, J3 V-, J4 Ex-I, J5 PG_Pins, J6 Exp, J7 VR-, J8 TX_RX_ES, J9 VR+, P1 CONN_01X08, P10 Analog, P3 DIO, P5 sen-cap, P7 NRF, Q1 MMBT3906, Q2 MMBT3904, Q3 MMBT3906, U1 MCP2200, U10 TL082, U11 6S21, U12 6S21, U13 TL082, U15 ESP8266, U16 TL082, U2 74HC126, U3 PIC24EP256GP204, U4 TC1240A, U5 7660, U6 LM1117-3.3, U7 LM324, U8 TL082, U9 MCP4728, X1 12MHz

Commit message: recheck all circuits and clean up fill zone by rerouting the nets using freerouting and manually
Connections:
- C1 pad 1: (no net) -> Vdd
- C1 pad 2: (no net) -> GND
- C10 pad 1: (no net) -> GND
- C11 pad 2: (no net) -> GND
- C12 pad 1: (no net) -> V+
- C12 pad 2: (no net) -> GND
- C13 pad 1: (no net) -> GND
- C13 pad 2: (no net) -> Vdd
- C15 pad 2: (no net) -> GND
- C17 pad 1: (no net) -> GND
- C18 pad 1: (no net) -> GND
- C19 pad 1: (no net) -> GND
- C19 pad 2: (no net) -> V-
- C2 pad 1: (no net) -> GND
- C2 pad 2: (no net) -> Vdd
- C20 pad 1: (no net) -> GND
- C20 pad 2: (no net) -> +5V
- C21 pad 1: (no net) -> Vdd
- C21 pad 2: (no net) -> GND
- C22 pad 1: (no net) -> GND
- C24 pad 1: (no net) -> GND
- C26 pad 1: (no net) -> GND
- C27 pad 2: (no net) -> GND
- C28 pad 1: (no net) -> GND
- C30 pad 1: (no net) -> SINE1
- C31 pad 1: (no net) -> GND
- C32 pad 2: (no net) -> GND
- C34 pad 1: (no net) -> GND
- C35 pad 1: (no net) -> GND
- C37 pad 1: (no net) -> GND
- C38 pad 1: (no net) -> GND
- C39 pad 1: (no net) -> GND
- C4 pad 1: (no net) -> Vdd
- C4 pad 2: (no net) -> GND
- C40 pad 2: (no net) -> GND
- C41 pad 1: (no net) -> GND
- C5 pad 1: (no net) -> Vdd
- C5 pad 2: (no net) -> GND
- C7 pad 2: (no net) -> GND
- C8 pad 1: (no net) -> GND
- C8 pad 2: (no net) -> 12MHz
- C9 pad 1: (no net) -> GND
- C9 pad 2: (no net) -> +5V
- CON1 pad 4: (no net) -> GND
- CON1 pad 5: (no net) -> GND
- CON1 pad 6: (no net) -> GND
- D1 pad 1: (no net) -> GND
- D2 pad 2: (no net) -> GND
- D3 pad 1: (no net) -> GND
- D4 pad 1: (no net) -> GND
- F1 pad 2: (no net) -> +5V
- J10 pad 1: (no net) -> SCL
- J11 pad 1: (no net) -> GND
- J11 pad 2: (no net) -> Vdd
- J12 pad 1: (no net) -> Vdd
- J12 pad 2: (no net) -> AN8
- J2 pad 1: (no net) -> GND
- J4 pad 1: (no net) -> GND
- J4 pad 2: (no net) -> /MCLR
- J5 pad 1: (no net) -> +5V
- J6 pad 1: (no net) -> SDI
- J6 pad 2: (no net) -> SDO
- J6 pad 3: (no net) -> SCK
- J8 pad 2: (no net) -> /RxD
- L1 pad 2: (no net) -> Vdd
- MH1 pad 1: (no net) -> GND
- MH3 pad 1: (no net) -> GND
- MH4 pad 1: (no net) -> GND
- P1 pad 5: (no net) -> GND
- P1 pad 6: (no net) -> SINE1
- P1 pad 7: (no net) -> GND
- P10 pad 2: (no net) -> GND
- P10 pad 4: (no net) -> GND
- P10 pad 6: (no net) -> GND
- P10 pad 7: (no net) -> CH3
- P10 pad 8: (no net) -> GND
- P3 pad 10: (no net) -> GND
- P5 pad 2: (no net) -> GND
- P5 pad 5: (no net) -> GND
- P5 pad 6: (no net) -> CH3.GAIN
- P7 pad 1: (no net) -> GND
- P7 pad 2: (no net) -> Vdd
- P7 pad 5: (no net) -> SCK
- P7 pad 6: (no net) -> SDI
- P7 pad 7: (no net) -> SDO
- R1 pad 1: (no net) -> Vdd
- R1 pad 2: (no net) -> /MCLR
- R17 pad 2: (no net) -> GND
- R2 pad 1: (no net) -> SCL
- R2 pad 2: (no net) -> Vdd
- R25 pad 1: (no net) -> GND
- R27 pad 2: (no net) -> GND
- R3 pad 2: (no net) -> Vdd
- R38 pad 1: (no net) -> CH3.GAIN
- R40 pad 2: (no net) -> GND
- R42 pad 2: (no net) -> SINE1
- R45 pad 1: (no net) -> GND
- R45 pad 2: (no net) -> CH3
- R53 pad 2: (no net) -> +5V
- R54 pad 1: (no net) -> /RxD
- R56 pad 2: (no net) -> /RxD
- R57 pad 2: (no net) -> /TxD
- RV1 pad 1: (no net) -> GND
- TP1 pad 1: (no net) -> +5V
- TP2 pad 1: (no net) -> Vdd
- U1 pad 1: (no net) -> Vdd
- U1 pad 17: (no net) -> Vdd
- U1 pad 2: (no net) -> 12MHz
- U1 pad 20: (no net) -> GND
- U10 pad 3: (no net) -> GND
- U11 pad 4: (no net) -> GND
- U11 pad 6: (no net) -> SDO
- U11 pad 7: (no net) -> SCK
- U12 pad 4: (no net) -> GND
- U12 pad 6: (no net) -> SDO
- U12 pad 7: (no net) -> SCK
- U13 pad 3: (no net) -> GND
- U13 pad 5: (no net) -> GND
- U13 pad 7: (no net) -> SINE1
- U15 pad 10: (no net) -> GND
- U15 pad 11: (no net) -> Vdd
- U15 pad 3: (no net) -> Vdd
- U15 pad 8: (no net) -> Vdd
- U15 pad 9: (no net) -> GND
- U16 pad 2: (no net) -> CH3.GAIN
- U16 pad 3: (no net) -> CH3
- U16 pad 5: (no net) -> GND
- U2 pad 1: (no net) -> +5V
- U2 pad 10: (no net) -> +5V
- U2 pad 13: (no net) -> +5V
- U2 pad 14: (no net) -> +5V
- U2 pad 4: (no net) -> +5V
- U2 pad 7: (no net) -> GND
- U3 pad 16: (no net) -> GND
- U3 pad 18: (no net) -> /MCLR
- U3 pad 27: (no net) -> AN8
- U3 pad 28: (no net) -> Vdd
- U3 pad 29: (no net) -> GND
- U3 pad 31: (no net) -> 12MHz
- U3 pad 33: (no net) -> SCL
- U3 pad 34: (no net) -> SDO
- U3 pad 35: (no net) -> SDI
- U3 pad 36: (no net) -> SCK
- U3 pad 39: (no net) -> GND
- U3 pad 40: (no net) -> Vdd
- U3 pad 43: (no net) -> /RxD
- U3 pad 6: (no net) -> GND
- U4 pad 1: (no net) -> +5V
- U4 pad 2: (no net) -> GND
- U4 pad 4: (no net) -> GND
- U5 pad 3: (no net) -> GND
- U6 pad 1: (no net) -> GND
- U6 pad 2: (no net) -> Vdd
- U6 pad 3: (no net) -> +5V
- U6 pad 4: (no net) -> Vdd
- U8 pad 3: (no net) -> GND
- U9 pad 10: (no net) -> GND
- U9 pad 2: (no net) -> SCL
- X1 pad 1: (no net) -> 12MHz
Routing:
- net GND: track 0.00 -> 545.6 mm, vias 0 -> 20
- net Vdd: track 0.00 -> 195.3 mm, vias 0 -> 7
- net +5V: track 0.00 -> 117.6 mm, vias 0 -> 6
- net SCK: track 0.00 -> 60.5 mm, vias 0 -> 1
- net SCL: track 0.00 -> 53.3 mm, vias 0 -> 2
- net SDO: track 0.00 -> 53.3 mm, vias 0 -> 1
- net 12MHz: track 0.00 -> 52.6 mm, vias 0 -> 1
- net SDI: track 0.00 -> 48.8 mm
- net /RxD: track 0.00 -> 37.7 mm, vias 0 -> 1
- net CH3: track 0.00 -> 25.7 mm
- net /MCLR: track 0.00 -> 17.7 mm, vias 0 -> 1
- net SINE1: track 0.00 -> 13.0 mm
- net CH3.GAIN: track 0.00 -> 11.3 mm
- net AN8: track 0.00 -> 8.02 mm
- net V+: track 93.0 -> 96.4 mm
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