File: PCBs/kitspace_Potentiometer_mount_4LED/processed.kicad_pcb (KiCad board)
At the start: 2 copper layers, 40 x 30 mm, 7 parts

Commit message: recheck all circuits and clean up fill zone by rerouting the nets using freerouting and manually
Connections:
- LED 1 pad 1: (no net) -> Net-(RV1-Pad1)
- LED 2 pad 1: (no net) -> Net-(RV2-Pad1)
- LED 3 pad 1: (no net) -> Net-(RV3-Pad1)
- LED 4 pad 1: (no net) -> Net-(RV4-Pad1)
