File: PCBs/kitspace_esp8266/processed.kicad_pcb (KiCad board)
At the start: 2 copper layers, 50 x 50 mm, 30 parts, among them J1 Screw_Terminal_1x02, J2 Screw_Terminal_1x03, P1 CONN_02X04, P2 CONN_01X03, P3 CONN_01X03, P4 CONN_01X03, P5 CONN_01X03, P6 CONN_01X03, U1 LD1117S33TR

Commit message: recheck all circuits and clean up fill zone by rerouting the nets using freerouting and manually
Connections:
- C1 pad 1: (no net) -> +3V3
- C3 pad 1: (no net) -> +3V3
- C3 pad 2: (no net) -> GND
- D1 pad 2: (no net) -> VCC
- J1 pad 1: (no net) -> VCC
- J2 pad 1: (no net) -> +3V3
- JP1 pad 1: (no net) -> VCC
- JP1 pad 2: (no net) -> +3V3
- P1 pad 5: (no net) -> /PROG
- P1 pad 6: (no net) -> /RST
- P1 pad 8: (no net) -> +3V3
- P3 pad 1: (no net) -> +3V3
- P4 pad 1: (no net) -> +3V3
- P5 pad 1: (no net) -> +3V3
- P6 pad 1: (no net) -> +3V3
- PROG1 pad 1: (no net) -> /PROG
- R1 pad 1: (no net) -> /RST
- R1 pad 2: (no net) -> +3V3
- R2 pad 2: (no net) -> +3V3
- R3 pad 1: (no net) -> +3V3
- REF** pad 1: (no net) -> +3V3 (x3)
- REF** pad 12: (no net) -> /PROG
- RESET1 pad 2: (no net) -> /RST
- U1 pad 2: (no net) -> +3V3
Routing:
- net +3V3: track 0.00 -> 133.8 mm
- net VCC: track 0.00 -> 46.5 mm
- net /RST: track 0.00 -> 44.8 mm
- net /PROG: track 0.00 -> 44.1 mm, vias 0 -> 3
- net GND: track 167.3 -> 178.4 mm

Commit message: clean psbc that are missed before
Parts:
- removed the REF** at (152.4, 83.8)
- removed the REF** at (137.2, 83.8)
- added REF**_5: Pin_Header_Straight_1x10, Pin_Headers:Pin_Header_Straight_1x10, F.Cu at (137.2, 83.8)
- added REF**_6: Pin_Header_Straight_1x12, Pin_Headers:Pin_Header_Straight_1x12, F.Cu at (152.4, 83.8)
- renumbered REF** to REF**_10, REF** to REF**_11, REF** to REF**_2, REF** to REF**_3, REF** to REF**_4, REF** to REF**_7, REF** to REF**_8, REF** to REF**_9
