File: PCBs/retroreflectors_SALSAFLOCK/processed.kicad_pcb (KiCad board)
At the start: 2 copper layers, 30.8 x 52.8 mm, 15 parts, among them J1 DB15-VGA, J2 DB15-VGA, P2 ANTENNA, Q1 MOSFET_N, Q2 MOSFET_N

Commit message: recheck all circuits and clean up fill zone by rerouting the nets using freerouting and manually
Connections:
- C1 pad 1: (no net) -> GND
- J1 pad 0: (no net) -> /SHIELD
- J2 pad 0: (no net) -> /SHIELD
- Q2 pad B: (no net) -> GND
- Q2 pad S: (no net) -> GND
Routing:
- net /SHIELD: track 0.00 -> 84.2 mm
- net GND: track 1.64 -> 15.1 mm
