File: PCBs/retroreflectors_TANGOFLOCK/processed.kicad_pcb (KiCad board)
At the start: 2 copper layers, 31.8 x 31.8 mm, 5 parts, among them J1 USB-DEVICE-SHIELD, J2 USB-DEVICE-SHIELD, P2 ANTENNA, Q1 MOSFET_N

Commit message: recheck all circuits and clean up fill zone by rerouting the nets using freerouting and manually
Connections:
- J1 pad 4: (no net) -> GND
- J1 pad 5: (no net) -> /SHIELD
- J2 pad 4: (no net) -> GND
- J2 pad 5: (no net) -> /SHIELD
Routing:
- net /SHIELD: track 0.00 -> 46.9 mm
- net GND: track 4.59 -> 26.1 mm
Other:
- board text removed: "20140728"
- board text removed: "TANGOFLOCK"
