File: PCBs/z2amiller_sensorboard_programmer/processed.kicad_pcb (KiCad board)
At the start: 2 copper layers, 26 x 18.4 mm, 8 parts, among them P2 CONN_01X06

Commit message: recheck all circuits and clean up fill zone by rerouting the nets using freerouting and manually
Connections:
- USB MODULE pad 2: (no net) -> Net-(P1-Pad2)
- USB MODULE pad 6: (no net) -> +5V
