File: PCBs/CPU-Power-Supply-Mod_CPU_Power_Supply_Mod/processed.kicad_pcb (KiCad board)
At the start: 2 copper layers, 38 parts, among them K1 RELAY_SPST, K2 RELAY_SPST, K3 RELAY_SPST, K4 RELAY_SPST, P1 ICSP, P2 ATX 2.x, P3 PWR OUT, P4 PG SWT, Q1 PN2907, Q2 PN2907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

Commit message: debug boundaries of PCBs
Other:
- board outline added: 150 x 70 mm
