File: PCBs/Practicas-Curso-Kicad_Ejercicio_2/processed.kicad_pcb (KiCad board)
At the start: 2 copper layers, 15 parts, among them J1 DB9, U1 AMIS42665TJAA1RG, U2 SP-232v2

Commit message: debug boundaries of PCBs
Other:
- board outline added: 40.6 x 60.9 mm
