File: PCBs/RoBoC_CameraAdaptor/processed.kicad_pcb (KiCad board)
At the start: 2 copper layers, 6 parts, among them P1 CONN_02X12, P2 CONN_02X09, U1 Oscillator

Commit message: debug boundaries of PCBs
Other:
- board outline added: 36.8 x 43.8 mm
Changed lines of the file:
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@@
   (general
     (thickness 1.6)
-    (drawings 4)
+    (drawings 8)
     (tracks 156)
     (zones 0)
@@
     (0 F.Cu signal)
     (31 B.Cu signal)
-    (32 B.Adhes user)
+    (32 B.Adhes user hide)
     (33 F.Adhes user hide)
-    (34 B.Paste user)
-    (35 F.Paste user)
-    (36 B.SilkS user)
-    (37 F.SilkS user)
-    (38 B.Mask user)
-    (39 F.Mask user)
-    (40 Dwgs.User user)
-    (41 Cmts.User user)
-    (42 Eco1.User user)
-    (43 Eco2.User user)
+    (34 B.Paste user hide)
+    (35 F.Paste user hide)
+    (36 B.SilkS user hide)
+    (37 F.SilkS user hide)
+    (38 B.Mask user hide)
+    (39 F.Mask user hide)
+    (40 Dwgs.User user hide)
+    (41 Cmts.User user hide)
+    (42 Eco1.User user hide)
+    (43 Eco2.User user hide)
     (44 Edge.Cuts user)
-    (45 Margin user)
-    (46 B.CrtYd user)
-    (47 F.CrtYd user)
-    (48 B.Fab user)
-    (49 F.Fab user)
+    (45 Margin user hide)
+    (46 B.CrtYd user hide)
+    (47 F.CrtYd user hide)
+    (48 B.Fab user hide)
+    (49 F.Fab user hide)
   )
   (setup
@@
       (effects (font (size 1 1) (thickness 0.15)) (justify mirror))
     )
+    (fp_line (start -3.3 1.15) (end 3.3 1.15) (layer B.CrtYd) (width 0.05))
+    (fp_line (start -3.3 -1.15) (end 3.3 -1.15) (layer B.CrtYd) (width 0.05))
+    (fp_line (start -3.3 1.15) (end -3.3 -1.15) (layer B.CrtYd) (width 0.05))
+    (fp_line (start 3.3 1.15) (end 3.3 -1.15) (layer B.CrtYd) (width 0.05))
+    (fp_line (start 1 1.025) (end -1 1.025) (layer B.SilkS) (width 0.15))
     (fp_line (start -1 -1.025) (end 1 -1.025) (layer B.SilkS) (width 0.15))
-    (fp_line (start 1 1.025) (end -1 1.025) (layer B.SilkS) (width 0.15))
-    (fp_line (start 3.3 1.15) (end 3.3 -1.15) (layer B.CrtYd) (width 0.05))
-    (fp_line (start -3.3 1.15) (end -3.3 -1.15) (layer B.CrtYd) (width 0.05))
-    (fp_line (start -3.3 -1.15) (end 3.3 -1.15) (layer B.CrtYd) (width 0.05))
-    (fp_line (start -3.3 1.15) (end 3.3 1.15) (layer B.CrtYd) (width 0.05))
     (pad 1 smd rect (at -2 0 270) (size 2 1.6) (layers B.Cu B.Paste B.Mask)
       (net 1 +3V3))
@@
       (effects (font (size 1 1) (thickness 0.15)))
     )
+    (fp_line (start -1.75 -1.75) (end -1.75 29.7) (layer F.CrtYd) (width 0.05))
+    (fp_line (start 4.3 -1.75) (end 4.3 29.7) (layer F.CrtYd) (width 0.05))
+    (fp_line (start -1.75 -1.75) (end 4.3 -1.75) (layer F.CrtYd) (width 0.05))
+    (fp_line (start -1.75 29.7) (end 4.3 29.7) (layer F.CrtYd) (width 0.05))
+    (fp_line (start 3.81 29.21) (end 3.81 -1.27) (layer F.SilkS) (width 0.15))
+    (fp_line (start -1.27 1.27) (end -1.27 29.21) (layer F.SilkS) (width 0.15))
+    (fp_line (start 3.81 29.21) (end -1.27 29.21) (layer F.SilkS) (width 0.15))
+    (fp_line (start 3.81 -1.27) (end 1.27 -1.27) (layer F.SilkS) (width 0.15))
+    (fp_line (start 0 -1.55) (end -1.55 -1.55) (layer F.SilkS) (width 0.15))
+    (fp_line (start 1.27 -1.27) (end 1.27 1.27) (layer F.SilkS) (width 0.15))
+    (fp_line (start 1.27 1.27) (end -1.27 1.27) (layer F.SilkS) (width 0.15))
     (fp_line (start -1.55 -1.55) (end -1.55 0) (layer F.SilkS) (width 0.15))
-    (fp_line (start 1.27 1.27) (end -1.27 1.27) (layer F.SilkS) (width 0.15))
-    (fp_line (start 1.27 -1.27) (end 1.27 1.27) (layer F.SilkS) (width 0.15))
-    (fp_line (start 0 -1.55) (end -1.55 -1.55) (layer F.SilkS) (width 0.15))
-    (fp_line (start 3.81 -1.27) (end 1.27 -1.27) (layer F.SilkS) (width 0.15))
-    (fp_line (start 3.81 29.21) (end -1.27 29.21) (layer F.SilkS) (width 0.15))
-    (fp_line (start -1.27 1.27) (end -1.27 29.21) (layer F.SilkS) (width 0.15))
-    (fp_line (start 3.81 29.21) (end 3.81 -1.27) (layer F.SilkS) (width 0.15))
-    (fp_line (start -1.75 29.7) (end 4.3 29.7) (layer F.CrtYd) (width 0.05))
-    (fp_line (start -1.75 -1.75) (end 4.3 -1.75) (layer F.CrtYd) (width 0.05))
-    (fp_line (start 4.3 -1.75) (end 4.3 29.7) (layer F.CrtYd) (width 0.05))
-    (fp_line (start -1.75 -1.75) (end -1.75 29.7) (layer F.CrtYd) (width 0.05))
     (pad 1 thru_hole rect (at 0 0 90) (size 1.7272 1.7272) (drill 1.016) (layers *.Cu *.Mask F.SilkS)
       (net 1 +3V3))
@@
       (effects (font (size 1 1) (thickness 0.15)))
     )
+    (fp_line (start -1.75 -1.75) (end -1.75 22.1) (layer F.CrtYd) (width 0.05))
+    (fp_line (start 4.3 -1.75) (end 4.3 22.1) (layer F.CrtYd) (width 0.05))
+    (fp_line (start -1.75 -1.75) (end 4.3 -1.75) (layer F.CrtYd) (width 0.05))
+    (fp_line (start -1.75 22.1) (end 4.3 22.1) (layer F.CrtYd) (width 0.05))
+    (fp_line (start 3.81 21.59) (end 3.81 -1.27) (layer F.SilkS) (width 0.15))
+    (fp_line (start -1.27 1.27) (end -1.27 21.59) (layer F.SilkS) (width 0.15))
+    (fp_line (start 3.81 21.59) (end -1.27 21.59) (layer F.SilkS) (width 0.15))
+    (fp_line (start 3.81 -1.27) (end 1.27 -1.27) (layer F.SilkS) (width 0.15))
+    (fp_line (start 0 -1.55) (end -1.55 -1.55) (layer F.SilkS) (width 0.15))
+    (fp_line (start 1.27 -1.27) (end 1.27 1.27) (layer F.SilkS) (width 0.15))
+    (fp_line (start 1.27 1.27) (end -1.27 1.27) (layer F.SilkS) (width 0.15))
     (fp_line (start -1.55 -1.55) (end -1.55 0) (layer F.SilkS) (width 0.15))
-    (fp_line (start 1.27 1.27) (end -1.27 1.27) (layer F.SilkS) (width 0.15))
-    (fp_line (start 1.27 -1.27) (end 1.27 1.27) (layer F.SilkS) (width 0.15))
-    (fp_line (start 0 -1.55) (end -1.55 -1.55) (layer F.SilkS) (width 0.15))
-    (fp_line (start 3.81 -1.27) (end 1.27 -1.27) (layer F.SilkS) (width 0.15))
-    (fp_line (start 3.81 21.59) (end -1.27 21.59) (layer F.SilkS) (width 0.15))
-    (fp_line (start -1.27 1.27) (end -1.27 21.59) (layer F.SilkS) (width 0.15))
-    (fp_line (start 3.81 21.59) (end 3.81 -1.27) (layer F.SilkS) (width 0.15))
-    (fp_line (start -1.75 22.1) (end 4.3 22.1) (layer F.CrtYd) (width 0.05))
-    (fp_line (start -1.75 -1.75) (end 4.3 -1.75) (layer F.CrtYd) (width 0.05))
-    (fp_line (start 4.3 -1.75) (end 4.3 22.1) (layer F.CrtYd) (width 0.05))
-    (fp_line (start -1.75 -1.75) (end -1.75 22.1) (layer F.CrtYd) (width 0.05))
     (pad 1 thru_hole rect (at 0 0 180) (size 1.7272 1.7272) (drill 1.016) (layers *.Cu *.Mask F.SilkS)
       (net 1 +3V3))
@@
       (effects (font (size 1 1) (thickness 0.15)) (justify mirror))
     )
+    (fp_line (start -3.3 1.2) (end 3.3 1.2) (layer B.CrtYd) (width 0.05))
+    (fp_line (start -3.3 -1.2) (end 3.3 -1.2) (layer B.CrtYd) (width 0.05))
+    (fp_line (start -3.3 1.2) (end -3.3 -1.2) (layer B.CrtYd) (width 0.05))
+    (fp_line (start 3.3 1.2) (end 3.3 -1.2) (layer B.CrtYd) (width 0.05))
+    (fp_line (start 1 -1.075) (end -1 -1.075) (layer B.SilkS) (width 0.15))
     (fp_line (start -1 1.075) (end 1 1.075) (layer B.SilkS) (width 0.15))
-    (fp_line (start 1 -1.075) (end -1 -1.075) (layer B.SilkS) (width 0.15))
-    (fp_line (start 3.3 1.2) (end 3.3 -1.2) (layer B.CrtYd) (width 0.05))
-    (fp_line (start -3.3 1.2) (end -3.3 -1.2) (layer B.CrtYd) (width 0.05))
-    (fp_line (start -3.3 -1.2) (end 3.3 -1.2) (layer B.CrtYd) (width 0.05))
-    (fp_line (start -3.3 1.2) (end 3.3 1.2) (layer B.CrtYd) (width 0.05))
     (pad 1 smd rect (at -2 0 90) (size 2 1.7) (layers B.Cu B.Paste B.Mask)
       (net 1 +3V3))
@@
       (effects (font (size 1 1) (thickness 0.15)) (justify mirror))
     )
+    (fp_line (start -3.3 1.2) (end 3.3 1.2) (layer B.CrtYd) (width 0.05))
+    (fp_line (start -3.3 -1.2) (end 3.3 -1.2) (layer B.CrtYd) (width 0.05))
+    (fp_line (start -3.3 1.2) (end -3.3 -1.2) (layer B.CrtYd) (width 0.05))
+    (fp_line (start 3.3 1.2) (end 3.3 -1.2) (layer B.CrtYd) (width 0.05))
+    (fp_line (start 1 -1.075) (end -1 -1.075) (layer B.SilkS) (width 0.15))
     (fp_line (start -1 1.075) (end 1 1.075) (layer B.SilkS) (width 0.15))
-    (fp_line (start 1 -1.075) (end -1 -1.075) (layer B.SilkS) (width 0.15))
-    (fp_line (start 3.3 1.2) (end 3.3 -1.2) (layer B.CrtYd) (width 0.05))
-    (fp_line (start -3.3 1.2) (end -3.3 -1.2) (layer B.CrtYd) (width 0.05))
-    (fp_line (start -3.3 -1.2) (end 3.3 -1.2) (layer B.CrtYd) (width 0.05))
-    (fp_line (start -3.3 1.2) (end 3.3 1.2) (layer B.CrtYd) (width 0.05))
     (pad 1 smd rect (at -2 0 90) (size 2 1.7) (layers B.Cu B.Paste B.Mask)
       (net 1 +3V3))
@@
       (effects (font (size 1 1) (thickness 0.15)) (justify mirror))
     )
+    (fp_line (start -3.5 2.5) (end 3.5 2.5) (layer B.SilkS) (width 0.15))
+    (fp_line (start 3.5 2.5) (end 3.5 -2.5) (layer B.SilkS) (width 0.15))
+    (fp_line (start 3.5 -2.5) (end -3.5 -2.5) (layer B.SilkS) (width 0.15))
     (fp_line (start -3.5 -2.5) (end -3.5 2.5) (layer B.SilkS) (width 0.15))
-    (fp_line (start 3.5 -2.5) (end -3.5 -2.5) (layer B.SilkS) (width 0.15))
-    (fp_line (start 3.5 2.5) (end 3.5 -2.5) (layer B.SilkS) (width 0.15))
-    (fp_line (start -3.5 2.5) (end 3.5 2.5) (layer B.SilkS) (width 0.15))
     (pad 1 smd rect (at -3.58 -2.8 90) (size 3.86 3.4) (layers B.Cu B.Paste B.Mask)
       (net 1 +3V3))
@@
       (net 1 +3V3))
   )
+  (gr_line (start 77.48016 118.09984) (end 77.48016 74.30008) (layer Edge.Cuts) (width 0.1))
+  (gr_line (start 114.29238 118.11508) (end 77.48016 118.09984) (layer Edge.Cuts) (width 0.1))
+  (gr_line (start 114.30762 74.30516) (end 114.29238 118.11508) (layer Edge.Cuts) (width 0.1))
+  (gr_line (start 77.48016 74.30008) (end 114.30762 74.30516) (layer Edge.Cuts) (width 0.1))
   (gr_line (start 77.47 118.11) (end 77.47 74.295) (angle 90) (layer Dwgs.User) (width 0.2))
   (gr_line (start 114.3 118.11) (end 77.47 118.11) (angle 90) (layer Dwgs.User) (width 0.2))
