File: PCBs/arduino-led-driver_arduino-led-driver/processed.kicad_pcb (KiCad board)
At the start: 2 copper layers, 118 parts, among them J1 CONN_01X02, J10 CONN_01X02, J11 CONN_01X02, J12 CONN_01X02, J13 CONN_01X02, J14 CONN_01X02, J15 CONN_01X02, J16 CONN_01X02, J17 CONN_01X02, J18 CONN_01X02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

Commit message: debug boundaries of PCBs
Other:
- board outline added: 70 x 44 mm
